Commit message: separated alg and env cfgs, added q-value critic to shac2, warp cartpole working

File: src/shac/envs/assets/cartpole.urdf (robot description, URDF)
Before this commit: robot physics, 3 links, 2 joints
Joints:
- joint cart_to_pole: origin xyz=0.0 0.0 0 -> xyz=0.0 0.0 0 rpy=0. 3.1415 0.

Commit message: Revert cartpole rotation

File: src/shac/envs/assets/cartpole.urdf (robot description, URDF)
Before this commit: robot physics, 3 links, 2 joints
Joints:
- joint cart_to_pole: origin xyz=0.0 0.0 0 rpy=0. 3.1415 0. -> xyz=0.0 0.0 0

Commit message: added mpc baseline

File: src/shac/envs/assets/cartpole.urdf (robot description, URDF)
Before this commit: robot physics, 3 links, 2 joints
Joints:
- joint cart_to_pole: origin xyz=0.0 0.0 0 rpy=0. 3.1415 0. -> xyz=0.0 0.0 0 rpy=0. 0. 0.
